File: Esquemático/V0.1.sch (EAGLE design)
At the start: 47 parts, among them IC1 7805T, IC2 MCP2515-I/P, IC3 MCP2551-I/P, IC4 7805T, K1 AQYAQY27, K2 AQYAQY27, Q1 20M

Commit message: Circuito Módulo expansão i/o CAN
tem MCP25050 e MCP2551
2 ENTRADAS E 6 SAIDAS
Parts:
- removed 12V: (no value), con-ptr500:AK300/2
- removed IC4: 7805T, linear:7805T
- added 24V, RELAY3, RELAY4, RELAY5, RELAY6: (no value), con-ptr500:AK300/2
- added C12, C31, C34: 100nF, rcl:C-EUC0805
- added C13: 100uF/50V, rcl:CPOL-EUE5-10.5
- added C14: 100uF/15V, rcl:CPOL-EUE5-10.5
- added C15, C30, C33: 10uF/15V, rcl:CPOL-EUE5-10.5
- added C16: 220uF/ESR, rcl:CPOL-EUE5-10.5
- added C17: 10nF, rcl:C-EUC0805
- added D10: SBL845/B340A, SparkFun-DiscreteSemi:DIODE-SCHOTTKY-B340A
- added D3, D4, D5, D6, D7, D8: 1N4933, diode:1N4933
- added D9: BZV85C33, diode:ZENER-DIODEF126-10
- added F1: 1A-Slow, special:FUSE
- added K3, K4, K5, K6: AQYAQY27, relay:AQYAQY27
- added L1: 15uH/22uH/3A, inductors:DR1030
- added L3: 22uH/5mA, inductors:BL01RN1A
- added LED10, LED11, LED12, LED13, LED14, LED9: (no value), led:LED3MM
- added OK1, OK2: LTV816, optocoupler:LTV816
- added R12, R14, R16, R18, R20, R23: 1K, rcl:R-EU_0204/5
- added R13, R15, R17, R19, R22, R25: 330, rcl:R-EU_0204/5
- added R21, R24: 510, rcl:R-EU_0204/5
- added R26: 10K/1%, rcl:R-EU_R0603
- added R27: 3K24/1%, rcl:R-EU_R0603
- added R28: 0R, rcl:R-EU_R0603
- added S1, S2: (no value), switch-omron:10-XX
- added U2: (no value), texas_tps5430:TPS5430DDAG4
- added U3: LM1117-3.3V, SparkFun-IC-Power:V_REG_LM1117SOT223
- C7: value (none) -> 100nF; device rcl:CPOL-EUE3.5-8 -> rcl:C-EUC0805
- C8: value (none) -> 100nF; device rcl:CPOL-EUE2.5-5 -> rcl:C-EUC0805
- D2: value 1N4004 -> 1N5400; device diode:1N4004 -> diode:1N5400
- R8, R9: value 10K -> 1K
Connections:
- removed net N$29 (its old number): K2.DS1, RELAY2-2.KL
- new net +3.3V: C12.1, C15.+, U3.OUT, U3.OUT@1
- new net AGND: C33.-, C34.2, R28.2
- new net GP2: R16.1, U$1.GP2/AN2/PWM1
- new net GP3: R9.1, U$1.GP3/AN3/PWM2
- new net GP4: R14.1, U$1.GP4/VREF-
- new net GP5: R18.1, U$1.GP5/VREF+
- new net GP6: OK1.EMIT, R20.1, U$1.GP6/CLKOUT
- new net GP7: OK2.EMIT, R23.1, U$1.GP7/~RST/VPP
- new net N$27: D3.A, RELAY1-2.KL
- new net N$30: D4.C, K2.DS1, LED8.C
- new net N$36: D4.A, RELAY2-2.KL
- new net N$37: K3.A, R12.2
- new net N$38: D5.C, K3.DS1, LED9.C
- new net N$39: K3.DS2, RELAY3-1.KL
- new net N$40: LED9.A, R13.2
- new net N$41: D5.A, RELAY3-2.KL
- new net N$42: K4.A, R14.2
- new net N$43: D6.C, K4.DS1, LED10.C
- new net N$44: K4.DS2, RELAY4-1.KL
- new net N$45: LED10.A, R15.2
- new net N$46: D6.A, RELAY4-2.KL
- new net N$47: K5.A, R16.2
- new net N$48: D7.C, K5.DS1, LED11.C
- new net N$49: K5.DS2, RELAY5-1.KL
- new net N$50: LED11.A, R17.2
- new net N$51: D7.A, RELAY5-2.KL
- new net N$52: K6.A, R18.2
- new net N$53: D8.C, K6.DS1, LED12.C
- new net N$54: K6.DS2, RELAY6-1.KL
- new net N$55: LED12.A, R19.2
- new net N$56: D8.A, RELAY6-2.KL
- new net N$57: R21.2, S1.P, S1.P1
- new net N$58: R24.2, S2.P, S2.P1
- new net N$59: OK1.A, R21.1
- new net N$60: LED13.A, R22.2
- new net N$61: OK1.C, R22.1
- new net N$62: OK2.A, R24.1
- new net N$63: LED14.A, R25.2
- new net N$64: OK2.C, R25.1
- new net N$65: C14.+, C16.+, C8.1, L1.2, U3.IN
- new net N$66: C17.2, U2.BOOT
- new net N$67: R26.2, R27.1, U2.VSENSE
- new net N$68: 24V-1.KL, D2.A
- new net VCC/2: C33.+, C34.1, L3.2
- net 5V: now also C17.1, C30.+, C31.1, D10.C, L1.1, L3.1, OK1.COL, OK2.COL, R13.1, R15.1, R17.1, R19.1, R26.1, S1.S, S1.S1, S2.S, S2.S1, U2.PH; no longer C8.+, IC4.VO
- net GND: now also 24V-2.KL, C12.2, C13.-, C14.-, C15.-, C16.-, C30.-, C31.2, C7.2, C8.2, D10.A, D9.A, K3.K, K4.K, K5.K, K6.K, LED13.C, LED14.C, R20.2, R23.2, R27.2, R28.1, U2.GND, U2.POWER_PAD, U3.ADJ; no longer 12V-2.KL, C7.-, C8.-, IC4.GND
- net GP0: no longer LED7.C
- net GP1: now also R12.1; no longer LED8.C, R9.1
- net N$21: now also C13.+, C7.1, D9.C, F1.2, U2.VIN; no longer 12V-1.KL, D2.A
- net N$23: now also F1.1; no longer C7.+, IC4.VI
- net N$26: now also D3.C, LED7.C; no longer RELAY1-2.KL
Other:
- note added: "ALIMENTAÇÃO 12/24/36v TO 5/3.3V"
- note added: "ENTRADAS A OPTOACOPLADORES"
- note added: "TRANSMISSÃO E CONVERSÃO DE CAN"
- moved on the sheet: C10, C11, C9, CAN-1, CAN-2, D2, K1, K2, LED5, LED6, LED7, LED8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

Commit message: alterado parte das saídas a rele
foi colocado 24v às saídas de rele, e o sinalizador na parte de comando
Parts:
- removed +12: 12V, con-ptr500:AK300/2
- removed C1: 470uF, rcl:CPOL-EUE3.5-8
- removed C2: 1uF, rcl:CPOL-EUE2.5-5
- removed C3, C6: 100n, rcl:C-EU050-025X075
- removed C4, C5: 15p, rcl:C-EU025-024X044
- removed D1: 1N4007, diode:1N4004
- removed D3, D4, D5, D6, D7, D8: 1N4933, diode:1N4933
- removed IC1: 7805T, linear:7805T
- removed IC2: MCP2515-I/P, MCP2515-IP:MCP2515-I/P
- removed IC3: MCP2551-I/P, MCP2551-IP:MCP2551-I/P
- removed LED10, LED11, LED12, LED9: (no value), led:LED3MM
- removed Q1: 20M, crystal:CRYSTALHC49S
- removed R15, R17, R19: 330, rcl:R-EU_0204/5
- removed R16, R18: 1K, rcl:R-EU_0204/5
- R1, R11, R13, R3: value 330 -> 510
- R12, R14, R9: value 1K -> 330
- R5: value 4.7k -> 510; device rcl:R-EU_0204/7 -> rcl:R-EU_0204/5
- R8: value 1K -> 510
Connections:
- removed net +5V: C2.+, C3.1, C6.2, IC1.VO, IC2.VDD, IC3.VDD, R1.2, R2.2, R3.1, R4.1
- removed net 0V: +12-2.KL, C1.-, C2.-, C4.1, C5.1, C6.1, IC1.GND, IC3.VSS, R5.2
- removed net N$10 (its old number): IC2.~CS
- removed net N$14 (its old number): C5.2, IC2.OSC2, Q1.2
- removed net N$18 (its old number): IC3.RS, R5.1
- removed net N$27 (its old number): D3.A, RELAY1-2.KL
- removed net N$29: K2.A, R9.2
- removed net N$3 (its old number): LED1.A, R1.1
- removed net N$30: D4.C, K2.DS1, LED8.C
- removed net N$35: LED8.A, R11.2
- removed net N$36: D4.A, RELAY2-2.KL
- removed net N$37: K3.A, R12.2
- removed net N$38: D5.C, K3.DS1, LED9.C
- removed net N$40: LED9.A, R13.2
- removed net N$41: D5.A, RELAY3-2.KL
- removed net N$42: K4.A, R14.2
- removed net N$43: D6.C, K4.DS1, LED10.C
- removed net N$45: LED10.A, R15.2
- removed net N$46: D6.A, RELAY4-2.KL
- removed net N$47: K5.A, R16.2
- removed net N$48: D7.C, K5.DS1, LED11.C
- removed net N$50: LED11.A, R17.2
- removed net N$51: D7.A, RELAY5-2.KL
- removed net N$52: K6.A, R18.2
- removed net N$53: D8.C, K6.DS1, LED12.C
- removed net N$55: LED12.A, R19.2
- removed net N$56: D8.A, RELAY6-2.KL
- removed net N$6 (its old number): IC2.~RX0BF, LED2.C
- removed net N$68: 24V-1.KL, D2.A
- new net 24V: 24V-1.KL, D2.A, K1.DS1, K2.DS1, K3.DS1, K4.DS1, K5.DS1, K6.DS1, RELAY1-2.KL, RELAY2-2.KL, RELAY3-2.KL, RELAY4-2.KL, RELAY5-2.KL, RELAY6-2.KL
- net 5V: no longer R10.1, R11.1, R13.1, R15.1, R17.1, R19.1
- net GND: now also LED1.C, LED2.C, LED3.C, LED4.C, LED7.C, LED8.C; no longer C3.2, IC2.VSS, K1.K, K2.K, K3.K, K4.K, K5.K, K6.K
- net GP1: now also R1.1; no longer R12.1
- net GP2: now also R3.1; no longer R16.1
- net GP3: now also R5.1; no longer R9.1
- net GP4: now also R11.1; no longer R14.1
- net GP5: now also R13.1; no longer R18.1
- net N$1: now also K1.K, R10.1; no longer +12-1.KL, D1.A
- net N$11: now also K2.A, R5.2; no longer IC2.SI
- net N$12: now also LED3.A, R9.2; no longer IC2.SCK
- net N$13: now also K2.K, R9.1; no longer IC2.SO
- net N$15: now also K4.A, R11.2; no longer C4.2, IC2.OSC1, Q1.1
- net N$16: now also LED4.A, R12.2; no longer LED3.A, R3.2
- net N$17: now also K4.K, R12.1; no longer LED4.A, R4.2
- net N$19: now also K6.A, R13.2; no longer IC3.CANL
- net N$2: now also K3.A, R1.2; no longer C1.+, D1.C, IC1.VI
- net N$20: now also LED8.A, R14.2; no longer IC3.CANH
- net N$26: now also K6.K, R14.1; no longer D3.C, K1.DS1, LED7.C
- net N$4: now also LED1.A, R2.2; no longer LED2.A, R2.1
- net N$5: now also K3.K, R2.1; no longer IC2.~RX1BF, LED1.C
- net N$7: now also K5.A, R3.2; no longer IC2.RXCAN, IC3.RXD, LED3.C
- net N$8: now also LED2.A, R4.2; no longer IC2.TXCAN, LED4.C
- net N$9: now also K5.K, R4.1; no longer IC2.~RESET
